Commit message: fix(stability): add front caster wheel to eliminate nose-dive tilt and map shaking, enable GUI by default

File: urdf/robot.urdf.xacro (robot description, xacro)
@@ -67,4 +67,23 @@
     <xacro:solid_sphere_inertia m="${caster_mass}" r="${caster_diameter/2}"/>
   </link>
+  <joint name="caster_front_joint" type="fixed">
+    <parent link="base_link"/>
+    <child link="caster_front_link"/>
+    <origin xyz="${base_diameter/2 - caster_inset} 0 ${caster_diameter/2 - floor_clearance}" rpy="0 0 0"/>
+  </joint>
+  <link name="caster_front_link">
+    <visual>
+      <geometry>
+        <sphere radius="${caster_diameter/2}"/>
+      </geometry>
+      <material name="grey"/>
+    </visual>
+    <collision>
+      <geometry>
+        <sphere radius="${caster_diameter/2}"/>
+      </geometry>
+    </collision>
+    <xacro:solid_sphere_inertia m="${caster_mass}" r="${caster_diameter/2}"/>
+  </link>
   <joint name="wheel_left_joint" type="continuous">
     <parent link="base_link"/>
@@ -176,4 +195,8 @@
     <mu2>0.001</mu2>
   </gazebo>
+  <gazebo reference="caster_front_link">
+    <mu1>0.001</mu1>
+    <mu2>0.001</mu2>
+  </gazebo>
   <gazebo reference="wheel_left_link">
     <mu1>1.0</mu1>
