Commit message: fix: obstacle bridging for chair legs, ball avoidance, bumper contact wiring, snappy rotation, and alcove coverage

File: urdf/plugins.xacro (robot description, xacro)
@@ -57,5 +57,5 @@
     <sensor name="bumper_left_contact" type="contact">
       <contact>
-        <collision>bumper_left_collision</collision>
+        <collision>base_footprint_fixed_joint_lump__bumper_left_collision_collision_1</collision>
         <topic>bumper_left</topic>
       </contact>
@@ -65,5 +65,5 @@
     <sensor name="bumper_right_contact" type="contact">
       <contact>
-        <collision>bumper_right_collision</collision>
+        <collision>base_footprint_fixed_joint_lump__bumper_right_collision_collision_2</collision>
         <topic>bumper_right</topic>
       </contact>
